Commit message: feat(major): modified structure

File: urdf/f16.urdf (robot description, URDF)
Before this commit: robot RobotAssembly_v2_10_cam_2, 19 links, 18 joints
Links:
- added link A_camera_link, mass 0.1; collision mesh filename=package://RobotAssembly_v2_10_cam_2/meshes/F_camera_link.STL; visual mesh filename=package://RobotAssembly_v2_10_cam_2/meshes/F_camera_link.STL
Joints:
- added joint A_camera_joint: type fixed, parent base_link, child A_camera_link, origin xyz=0.24 0 0.12 rpy=-1.5707963267949 0 -1.5707963267949
