Commit message: feat(tf): add robot state publisher

File: resources/urdf/f16.urdf (robot description, URDF)
Before this commit: robot RobotAssembly_v2_10_cam_2, 20 links, 19 joints
Links:
- added link livox_frame, mass 0.1
Joints:
- added joint livox_joint: type fixed, parent A_camera_link, child livox_frame, origin xyz=-0.08 0 0 rpy=0 0 0

Commit message: feat: bug fix and add point_lio

File: resources/urdf/f16.urdf (robot description, URDF)
Before this commit: robot RobotAssembly_v2_10_cam_2, 21 links, 20 joints
Joints:
- joint livox_joint: origin xyz=-0.08 0 0 rpy=0 0 0 -> xyz=0.24 0 0.20 rpy=0 0 0; parent A_camera_link -> base_link

Commit message: feat(urdf): add base_footprint

File: resources/urdf/f16.urdf (robot description, URDF)
Before this commit: robot RobotAssembly_v2_10_cam_2, 21 links, 20 joints
Links:
- added link base_footprint
Joints:
- added joint base_footprint_joint: type fixed, parent base_footprint, child base_link, origin xyz=0 0 0.5 rpy=0 0 0

File: resources/urdf/f8.urdf (robot description, URDF)
Before this commit: robot RobotAssembly_v3_1_3, 10 links, 9 joints
Links:
- added link base_footprint
Joints:
- added joint base_footprint_joint: type fixed, parent base_footprint, child base_link, origin xyz=0 0 0.5 rpy=0 0 0
