Commit message: feat(nav): adding navigation

File: resources/urdf/f16.urdf (robot description, URDF)
Before this commit: robot RobotAssembly_v2_10_cam_2, 22 links, 21 joints
Links:
- removed link livox_frame
- added link lidar_link, mass 0.1
Joints:
- joint livox_joint: child livox_frame -> lidar_link
