Commit message: feat(height_map): changed logic

File: resources/urdf/f4.urdf (robot description, URDF)
Before this commit: robot 2WL_V3_Assem_v2, 13 links, 12 joints
Links:
- added link A_camera_link, mass 0.0457681807749963; collision mesh filename=package://2WL_V3_Assem_v3/meshes/A_camera_link.STL; visual mesh filename=package://2WL_V3_Assem_v3/meshes/A_camera_link.STL
- added link F_camera_link, mass 0.0457682375319545; collision mesh filename=package://2WL_V3_Assem_v3/meshes/F_camera_link.STL; visual mesh filename=package://2WL_V3_Assem_v3/meshes/F_camera_link.STL
- added link lidar_link, mass 0.0523970418812064; collision mesh filename=package://2WL_V3_Assem_v3/meshes/lidar_link.STL; visual mesh filename=package://2WL_V3_Assem_v3/meshes/lidar_link.STL
- added link sensor_mount_link, mass 0.611294472871864; collision mesh filename=package://2WL_V3_Assem_v3/meshes/sensor_mount_link.STL; visual mesh filename=package://2WL_V3_Assem_v3/meshes/sensor_mount_link.STL
- link FL_caster_link: geometry collision mesh filename=package://2WL_V3_Assem_v3/meshes/FL_caster_link.STL; visual mesh filename=package://2WL_V3_Assem_v3/meshes/FL_caster_link.STL
- link FR_cater_link: geometry collision mesh filename=package://2WL_V3_Assem_v3/meshes/FR_cater_link.STL; visual mesh filename=package://2WL_V3_Assem_v3/meshes/FR_cater_link.STL
- link RL_caster_link: geometry collision mesh filename=package://2WL_V3_Assem_v3/meshes/RL_caster_link.STL; visual mesh filename=package://2WL_V3_Assem_v3/meshes/RL_caster_link.STL
- link RR_caster_link: geometry collision mesh filename=package://2WL_V3_Assem_v3/meshes/RR_caster_link.STL; visual mesh filename=package://2WL_V3_Assem_v3/meshes/RR_caster_link.STL
- link base_link: geometry collision mesh filename=package://2WL_V3_Assem_v3/meshes/base_link.STL; visual mesh filename=package://2WL_V3_Assem_v3/meshes/base_link.STL
- link left_leg_link: geometry collision mesh filename=package://2WL_V3_Assem_v3/meshes/left_leg_link.STL; visual mesh filename=package://2WL_V3_Assem_v3/meshes/left_leg_link.STL
- link left_shoulder_link: geometry collision mesh filename=package://2WL_V3_Assem_v3/meshes/left_shoulder_link.STL; visual mesh filename=package://2WL_V3_Assem_v3/meshes/left_shoulder_link.STL
- link left_upper_link: geometry collision mesh filename=package://2WL_V3_Assem_v3/meshes/left_upper_link.STL; visual mesh filename=package://2WL_V3_Assem_v3/meshes/left_upper_link.STL
- link left_wheel_link: geometry collision mesh filename=package://2WL_V3_Assem_v3/meshes/left_wheel_link.STL; visual mesh filename=package://2WL_V3_Assem_v3/meshes/left_wheel_link.STL
- link right_leg_link: geometry collision mesh filename=package://2WL_V3_Assem_v3/meshes/right_leg_link.STL; visual mesh filename=package://2WL_V3_Assem_v3/meshes/right_leg_link.STL
- link right_shoulder_link: geometry collision mesh filename=package://2WL_V3_Assem_v3/meshes/right_shoulder_link.STL; visual mesh filename=package://2WL_V3_Assem_v3/meshes/right_shoulder_link.STL
- link right_upper_link: geometry collision mesh filename=package://2WL_V3_Assem_v3/meshes/right_upper_link.STL; visual mesh filename=package://2WL_V3_Assem_v3/meshes/right_upper_link.STL
- link right_wheel_link: geometry collision mesh filename=package://2WL_V3_Assem_v3/meshes/right_wheel_link.STL; visual mesh filename=package://2WL_V3_Assem_v3/meshes/right_wheel_link.STL
Joints:
- added joint A_camera_joint: type fixed, parent sensor_mount_link, child A_camera_link, origin xyz=0.062914 0.0012578 -0.0175 rpy=-1.5708 0 -1.5708, axis 0 0 0
- added joint F_camera_joint: type fixed, parent sensor_mount_link, child F_camera_link, origin xyz=0.053264 0.0012578 -0.057725 rpy=-2.3562 0 -1.5708, axis 0 0 0
- added joint lidar_joint: type fixed, parent sensor_mount_link, child lidar_link, origin xyz=0.016496 0.00062477 0.0453 rpy=3.1416 0 0, axis 0 0 0
- added joint sensor_mount_joint: type fixed, parent base_link, child sensor_mount_link, origin xyz=0.021839 0.00099604 0.093686 rpy=0 0 0, axis 0 0 0
